File: pcb/split_EC_left.kicad_pcb (KiCad board)
At the start: 2 copper layers, 85 x 70 mm, 25 parts, among them J1 AE-USB2.0-TYPE-C, J2 AVR-ISP-6, J3 DF15(3.2)-20DP-0.65V(56), J4 TRRS jack, SW1 SW_Push, U1 BeetleUSB_with_USB, U2 74LS138

Commit message: Update pcb designs to rev.1
Parts:
- moved R4 2.08 mm to (143.0, 61.4), turned to 90 degrees
- moved R3 0.84 mm to (139.9, 61.4), turned to 90 degrees
Connections:
- R3 pad 1: SCL -> VCC
- R3 pad 2: GND -> SCL
- R4 pad 1: SDA -> VCC
- R4 pad 2: GND -> SDA
Routing:
- net VCC: track 109.6 -> 129.5 mm
- net GND: track 1.30 -> 13.5 mm, vias 224 -> 205
- net DATA: track 41.9 -> 35.1 mm
- net SCL: track 31.0 -> 35.2 mm
- net COL_A: track 100.1 -> 97.4 mm
- net SDA: track 33.0 -> 35.0 mm
- net ~RST: track 66.3 -> 65.0 mm
- net COL_B: track 90.9 -> 89.6 mm
- net COL_C: track 93.0 -> 94.3 mm
- net COL_3: track 24.3 -> 23.2 mm
- net COL_1: track 24.2 -> 23.2 mm
- net KEY: track 49.2 -> 50.1 mm
- net ENABLE: track 72.9 -> 73.7 mm
- net ROW_C: track 65.2 -> 64.5 mm
- net AVCC: track 53.9 -> 54.4 mm
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Other:
- board text added: "split EC left side rev.1 © B-SAKATU 2019"
- board text removed: "split EC left side rev. 0.1 © B-SAKATU 2019"
