File: pcb/split_EC_right.kicad_pcb (KiCad board)
At the start: 2 copper layers, 85 x 70 mm, 25 parts, among them J1 AE-USB2.0-TYPE-C, J2 AVR-ISP-6, J3 DF15(3.2)-20DP-0.65V(56), J4 TRRS jack, SW1 SW_Push, U1 BeetleUSB_with_USB, U2 74LS138

Commit message: Update pcb designs to rev.1
Parts:
- moved R4 2.08 mm to (84.5, 66.7), turned to 90 degrees
- moved R3 0.83 mm to (81.4, 66.7), turned to 90 degrees
Connections:
- R3 pad 1: SCL -> VCC
- R3 pad 2: GND -> SCL
- R4 pad 1: SDA -> VCC
- R4 pad 2: GND -> SDA
Routing:
- net AVCC: track 28.7 -> 46.7 mm
- net VCC: track 124.7 -> 140.0 mm
- net GND: track 1.95 -> 16.3 mm, vias 222 -> 225
- net SCL: track 24.2 -> 31.6 mm
- net COL_3: track 25.9 -> 21.4 mm
- net DATA: track 30.3 -> 26.4 mm
- net COL_C: track 66.1 -> 63.8 mm
- net ENABLE: track 92.9 -> 90.6 mm
- net PREV: track 74.6 -> 72.7 mm
- net SDA: track 25.9 -> 27.6 mm
- net ROW_B: track 83.2 -> 84.3 mm
- net COL_1: track 23.6 -> 22.6 mm
- net ~RST: track 67.5 -> 68.4 mm
- net Net-(J4-PadT): track 11.7 -> 12.6 mm
- net COL_B: track 61.1 -> 61.9 mm
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Other:
- board text added: "split EC right side rev.1 © B-SAKATU 2019"
- board text removed: "split EC right side rev. 0.1 © B-SAKATU 2019"
